Commit message: added everything up to part 3

File: mentorpi_description/urdf/mecanum.xacro (robot description, xacro)
@@ -54,10 +54,8 @@
       </material>
     </visual>
-    <collision>
-      <origin rpy="0 0 0" xyz="0 0 0"/>
-      <geometry>
-        <mesh filename="package://mentorpi_description/meshes/mecanum/wheel_lf_Link.STL"/>
-      </geometry>
-    </collision>
+<collision>
+  <origin rpy="1.5708 0 0" xyz="0 -0.0074 0"/>
+  <geometry><cylinder radius="0.0325" length="0.0344"/></geometry>
+</collision>
   </link>
   <joint name="wheel_lf_Joint" type="continuous">
@@ -82,10 +80,8 @@
       </material>
     </visual>
-    <collision>
-      <origin rpy="0 0 0" xyz="0 0 0"/>
-      <geometry>
-        <mesh filename="package://mentorpi_description/meshes/mecanum/wheel_rf_Link.STL"/>
-      </geometry>
-    </collision>
+<collision>
+  <origin rpy="0 0 0" xyz="0.0029 0 0.0113"/>
+  <geometry><box size="0.2119 0.1 0.0924"/></geometry>
+</collision>
   </link>
   <joint name="wheel_rf_Joint" type="continuous">
@@ -110,10 +106,8 @@
       </material>
     </visual>
-    <collision>
-      <origin rpy="0 0 0" xyz="0 0 0"/>
-      <geometry>
-        <mesh filename="package://mentorpi_description/meshes/mecanum/wheel_lb_Link.STL"/>
-      </geometry>
-    </collision>
+<collision>
+  <origin rpy="0 0 0" xyz="0.0029 0 0.0113"/>
+  <geometry><box size="0.2119 0.1 0.0924"/></geometry>
+</collision>
   </link>
   <joint name="wheel_lb_Joint" type="continuous">
@@ -138,10 +132,8 @@
       </material>
     </visual>
-    <collision>
-      <origin rpy="0 0 0" xyz="0 0 0"/>
-      <geometry>
-        <mesh filename="package://mentorpi_description/meshes/mecanum/wheel_rb_Link.STL"/>
-      </geometry>
-    </collision>
+<collision>
+  <origin rpy="0 0 0" xyz="0.0029 0 0.0113"/>
+  <geometry><box size="0.2119 0.1 0.0924"/></geometry>
+</collision>
   </link>
   <joint name="wheel_rb_Joint" type="continuous">
@@ -166,10 +158,8 @@
       </material>
     </visual>
-    <collision>
-      <origin rpy="0 0 0" xyz="0 0 0"/>
-      <geometry>
-        <mesh filename="package://mentorpi_description/meshes/mecanum/cam_Link.STL"/>
-      </geometry>
-    </collision>
+<collision>
+  <origin rpy="0 0 0" xyz="0.0029 0 0.0113"/>
+  <geometry><box size="0.2119 0.1 0.0924"/></geometry>
+</collision>
   </link>
   <joint name="cam_Joint" type="fixed">
@@ -194,10 +184,8 @@
       </material>
     </visual>
-    <collision>
-      <origin rpy="0 0 0" xyz="0 0 0"/>
-      <geometry>
-        <mesh filename="package://mentorpi_description/meshes/mecanum/lidar_Link.STL"/>
-      </geometry>
-    </collision>
+<collision>
+  <origin rpy="0 0 0" xyz="0.0029 0 0.0113"/>
+  <geometry><box size="0.2119 0.1 0.0924"/></geometry>
+</collision>
   </link>
   <joint name="lidar_Joint" type="fixed">

Commit message: Lab 7 Complete

File: mentorpi_description/urdf/mecanum.xacro (robot description, xacro)
@@ -54,8 +54,8 @@
       </material>
     </visual>
-<collision>
-  <origin rpy="1.5708 0 0" xyz="0 -0.0074 0"/>
-  <geometry><cylinder radius="0.0325" length="0.0344"/></geometry>
-</collision>
+    <collision>
+      <origin rpy="1.5708 0 0" xyz="0 -0.0074 0"/>
+      <geometry><cylinder radius="0.0325" length="0.0344"/></geometry>
+    </collision>
   </link>
   <joint name="wheel_lf_Joint" type="continuous">
@@ -80,8 +80,8 @@
       </material>
     </visual>
-<collision>
-  <origin rpy="0 0 0" xyz="0.0029 0 0.0113"/>
-  <geometry><box size="0.2119 0.1 0.0924"/></geometry>
-</collision>
+    <collision>
+      <origin rpy="1.5708 0 0" xyz="0 0.0074 0"/>
+      <geometry><cylinder radius="0.0325" length="0.0344"/></geometry>
+    </collision>
   </link>
   <joint name="wheel_rf_Joint" type="continuous">
@@ -106,8 +106,8 @@
       </material>
     </visual>
-<collision>
-  <origin rpy="0 0 0" xyz="0.0029 0 0.0113"/>
-  <geometry><box size="0.2119 0.1 0.0924"/></geometry>
-</collision>
+    <collision>
+      <origin rpy="1.5708 0 0" xyz="0 -0.0074 0"/>
+      <geometry><cylinder radius="0.0325" length="0.0344"/></geometry>
+    </collision>
   </link>
   <joint name="wheel_lb_Joint" type="continuous">
@@ -132,8 +132,8 @@
       </material>
     </visual>
-<collision>
-  <origin rpy="0 0 0" xyz="0.0029 0 0.0113"/>
-  <geometry><box size="0.2119 0.1 0.0924"/></geometry>
-</collision>
+    <collision>
+      <origin rpy="1.5708 0 0" xyz="0 0.0074 0"/>
+      <geometry><cylinder radius="0.0325" length="0.0344"/></geometry>
+    </collision>
   </link>
   <joint name="wheel_rb_Joint" type="continuous">
@@ -158,8 +158,8 @@
       </material>
     </visual>
-<collision>
-  <origin rpy="0 0 0" xyz="0.0029 0 0.0113"/>
-  <geometry><box size="0.2119 0.1 0.0924"/></geometry>
-</collision>
+    <collision>
+      <origin rpy="0 0 0" xyz="0.0029 0 0.0113"/>
+      <geometry><box size="0.2119 0.1 0.0924"/></geometry>
+    </collision>
   </link>
   <joint name="cam_Joint" type="fixed">
@@ -184,8 +184,8 @@
       </material>
     </visual>
-<collision>
-  <origin rpy="0 0 0" xyz="0.0029 0 0.0113"/>
-  <geometry><box size="0.2119 0.1 0.0924"/></geometry>
-</collision>
+    <collision>
+      <origin rpy="0 0 0" xyz="0.0029 0 0.0113"/>
+      <geometry><box size="0.2119 0.1 0.0924"/></geometry>
+    </collision>
   </link>
   <joint name="lidar_Joint" type="fixed">
